Commit message: backup

File: assets/RobotBimanualV4/urdf/RobotBimanualV4_gripper.urdf (robot description, URDF)
Before this commit: robot RobotBimanualV4, 18 links, 17 joints
Links:
- added link left_tool
- added link right_tool
Joints:
- added joint left_tool_joint: type fixed, parent link6, child left_tool, origin xyz=0 0.125 0 rpy=0 0 0
- added joint right_tool_joint: type fixed, parent link12, child right_tool, origin xyz=0 0.125 0 rpy=0 0 0

Commit message: Finish pick, curling and penholder test

File: assets/RobotBimanualV4/urdf/RobotBimanualV4_gripper.urdf (robot description, URDF)
Before this commit: robot RobotBimanualV4, 20 links, 19 joints
Joints:
- joint left_tool_joint: origin xyz=0 0.125 0 rpy=0 0 0 -> xyz=0 0.125 -0.015 rpy=0 0 0
- joint right_tool_joint: origin xyz=0 0.125 0 rpy=0 0 0 -> xyz=0 0.125 -0.015 rpy=0 0 0
